File: schema/eq5drive/eq5drive.sch (KiCad schematic (older format))
At the start: 3 parts

Commit message: Ajout des schemas
Parts:
- added C1, C2: 100n, Capacitor_THT:C_Disc_D3.0mm_W1.6mm_P2.50mm, symbol Device:C_Small
- added C3, C4: 100u, Capacitor_THT:CP_Axial_L10.0mm_D6.0mm_P15.00mm_Horizontal, symbol Device:CP_Small
- added J1, J3: Conn_01x04, Connector_PinHeader_2.54mm:PinHeader_1x04_P2.54mm_Vertical, symbol Connector_Generic:Conn_01x04
- added J2: Conn_01x05, Connector_PinHeader_2.54mm:PinHeader_1x05_P2.54mm_Vertical, symbol Connector_Generic:Conn_01x05
- A1, A2: renamed from A?; value Pololu_Breakout_A4988 -> A4988
- XA1: renamed from XA?; footprint (none) -> arduino-shield:mega-shield
Connections:
- net +5V: now reaches XA1.5V1 (5V)
- net +5V: now also A1.2 (VDD), A2.2 (VDD), XA1.5V3 (5V), XA1.5V4 (5V), C1.1, C2.1, J2.4 (Pin_4)
- net at XA1.A0: now also J2.1 (Pin_1)
- net at XA1.A1: now also J2.2 (Pin_2)
- net A10: now reaches XA1.A10
- net A10: now also A1.10 (MS1)
- net A11: now reaches XA1.A11
- net A11: now also A1.11 (MS2)
- net A12: now reaches XA1.A12
- net A12: now also A1.12 (MS3)
- net A13: now reaches XA1.A13
- net A13: now also A1.13 (~RESET)
- net A14: now reaches XA1.A14
- net A14: now also A1.15 (STEP)
- net A15: now reaches XA1.A15
- net A15: now also A1.16 (DIR)
- net A9: now reaches XA1.A9
- net A9: now also A1.9 (~ENABLE)
- net 10: now reaches XA1.D10
- net 10: now also A2.12 (MS3)
- net 11: now reaches XA1.D11
- net 11: now also A2.13 (~RESET)
- net 12: now reaches XA1.D12
- net 12: now also A2.15 (STEP)
- net 13: now reaches XA1.D13
- net 13: now also A2.16 (DIR)
- net at XA1.D2 (D2_INT0): now also J2.3 (Pin_3)
- net 7: now reaches XA1.D7
- net 7: now also A2.9 (~ENABLE)
- net 8: now reaches XA1.D8
- net 8: now also A2.10 (MS1)
- net 9: now reaches XA1.D9
- net 9: now also A2.11 (MS2)
- net GND: now reaches XA1.GND1 (GND)
- net GND: now also A1.1 (GND), A1.7 (GND), A2.1 (GND), A2.7 (GND), XA1.GND2 (GND), XA1.GND3 (GND), XA1.GND5 (GND), XA1.GND6 (GND), C1.2, C2.2, C3.2, C4.2, J2.5 (Pin_5)
- net Vdrive: now reaches XA1.VIN
- net Vdrive: now also A1.8 (VMOT), A2.8 (VMOT), C3.1, C4.1
- net at A1.3 (1B): now also J1.3 (Pin_3)
- net at A1.4 (1A): now also J1.2 (Pin_2)
- net at A1.5 (2A): now also J1.4 (Pin_4)
- net at A1.6 (2B): now also J1.1 (Pin_1)
- net at A2.3 (1B): now also J3.3 (Pin_3)
- net at A2.4 (1A): now also J3.2 (Pin_2)
- net at A2.5 (2A): now also J3.4 (Pin_4)
- net at A2.6 (2B): now also J3.1 (Pin_1)
- no-connect marks 0 -> 67
Other:
- note added: "Ascension droite"
- note added: "Declinaison"
- note added: "Joystick\n"
- moved on the sheet: A1, A2, XA1
