File: schema/schema-1.0.kicad_pcb (KiCad board)
At the start: 2 copper layers, 91.4 x 55.9 mm, 16 parts, among them J1 Conn_01x04_Male, J2 Conn_01x04_Male, J3 Conn_01x05_Male

Commit message: 2 version de projet kicad  v1.0  v2.0
Parts:
- moved G1 47.0 mm to (146.1, 74.9)
- moved A2 36.9 mm to (115.6, 86.4)
- moved C4 28.2 mm to (139.7, 81.3)
- moved C3 27.7 mm to (118.1, 95.2)
- moved C1 27.3 mm to (165.1, 83.8)
- moved J2 25.9 mm to (132.1, 96.5), turned to 180 degrees
- moved J3 23.9 mm to (106.7, 105.4)
- moved J1 23.6 mm to (151.1, 82.5), turned to 0 degrees
- moved C2 20.7 mm to (143.4, 95.2)
- moved G0 9.16 mm to (100.3, 73.7)
- moved A1 2.54 mm to (167.6, 94.0)
Routing:
- net +5V: track 0.00 -> 96.2 mm
- net +12V: track 0.00 -> 55.9 mm
- net Net-(J3-Pad5): track 0.00 -> 46.8 mm
- net Net-(J3-Pad4): track 0.00 -> 33.8 mm
- net Net-(J3-Pad3): track 0.00 -> 29.9 mm
- net Net-(A1-Pad3): track 0.00 -> 13.7 mm
- net Net-(A1-Pad4): track 0.00 -> 13.7 mm
- net Net-(A1-Pad5): track 0.00 -> 13.7 mm
- net Net-(A1-Pad6): track 0.00 -> 13.0 mm
- net /10: track 0.00 -> 12.8 mm
- net /9: track 0.00 -> 12.8 mm
- net /11: track 0.00 -> 12.8 mm
- net /8: track 0.00 -> 12.7 mm
- net Net-(A2-Pad3): track 0.00 -> 11.8 mm
- net Net-(A2-Pad4): track 0.00 -> 11.8 mm
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