File: schema/schema-2.0.kicad_pcb (KiCad board)
At the start: 2 copper layers, 91.4 x 55.9 mm, 16 parts, among them J1 Conn_01x04_Male, J2 Conn_01x04_Male, J3 Conn_01x05_Male

Commit message: 2 version de projet kicad  v1.0  v2.0
Parts:
- moved G1 47.0 mm to (99.1, 74.9)
- moved A2 36.9 mm to (152.4, 87.6)
- moved C4 28.2 mm to (143.5, 109.2)
- moved C3 27.7 mm to (144.8, 87.6)
- moved C1 27.3 mm to (139.8, 94.0)
- moved J2 25.9 mm to (137.2, 71.1), turned to 270 degrees
- moved J3 23.9 mm to (128.3, 95.1)
- moved J1 23.6 mm to (137.2, 101.6), turned to 270 degrees
- moved C2 20.7 mm to (147.3, 74.9)
- moved G0 9.16 mm to (105.4, 81.3)
- moved A1 2.54 mm to (170.2, 94.0)
Routing:
- net /10: track 12.8 -> 66.4 mm
- net /12: track 11.0 -> 49.0 mm
- net /11: track 12.8 -> 50.1 mm
- net /9: track 12.8 -> 50.1 mm
- net /13: track 11.0 -> 48.3 mm
- net /8: track 12.7 -> 49.8 mm
- net /7: track 11.8 -> 48.6 mm
- net +12V: track 55.9 -> 87.1 mm
- net Net-(A2-Pad6): track 11.7 -> 34.9 mm
- net Net-(J3-Pad5): track 46.8 -> 23.9 mm
- net +5V: track 96.2 -> 73.9 mm
- net Net-(A1-Pad3): track 13.7 -> 35.1 mm
- net Net-(A2-Pad5): track 11.8 -> 32.1 mm
- net Net-(A1-Pad4): track 13.7 -> 30.8 mm
- net Net-(A2-Pad4): track 11.8 -> 28.5 mm
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