File: schema/schema-2.2.kicad_pcb (KiCad board)
At the start: 2 copper layers, 91.4 x 55.9 mm, 16 parts, among them J1 Conn_01x04_Male, J2 Conn_01x04_Male, J3 Conn_01x05_Male

Commit message: Nouvelle version Version  : 1.0 2.0 2.2 2.3
Parts:
- J1, J2: footprint Connector_JST:JST_XH_B4B-XH-A_1x04_P2.50mm_Vertical -> Connector_JST:JST_XH_S4B-XH-A-1_1x04_P2.50mm_Horizontal
- J3: footprint Connector_JST:JST_XH_B5B-XH-A_1x05_P2.50mm_Vertical -> Connector_JST:JST_XH_S5B-XH-A-1_1x05_P2.50mm_Horizontal
- moved J3 10.7 mm to (132.1, 85.1), turned to 270 degrees
- moved C4 7.62 mm to (143.5, 101.6)
- moved C2 6.35 mm to (147.3, 81.3)
- moved J1 5.08 mm to (132.1, 101.6)
- moved J2 5.08 mm to (132.1, 71.1)
Connections:
- net Net-(J3-Pad3) renamed /A0
- net Net-(J3-Pad4) renamed /A1
- J3 pad 5: Net-(J3-Pad5) -> /A2
- SH1 pad 2: Net-(J3-Pad5) -> Net-(SH1-Pad2)
- SH1 pad A2: Net-(SH1-PadA2) -> /A2
Routing:
- net Net-(J3-Pad5): track 23.9 -> 0.00 mm
- net /A2: track 0.00 -> 20.8 mm
- net +12V: track 87.1 -> 70.6 mm
- net /10: track 66.4 -> 50.1 mm
- net /A1: track 34.8 -> 24.3 mm
- net Net-(A1-Pad5): track 27.2 -> 33.0 mm
- net Net-(A1-Pad4): track 30.8 -> 36.6 mm
- net Net-(A1-Pad6): track 23.6 -> 28.7 mm
- net Net-(A2-Pad6): track 34.9 -> 40.0 mm
- net Net-(A1-Pad3): track 35.1 -> 40.1 mm
- net Net-(A2-Pad5): track 32.1 -> 36.4 mm
- net Net-(A2-Pad4): track 28.5 -> 32.9 mm
- net Net-(A2-Pad3): track 24.9 -> 29.3 mm
- net /A0: track 27.3 -> 25.5 mm
- net +5V: track 73.9 -> 75.3 mm
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